File: pcb/machine-filter/main-cv-inputs-1-4.kicad_sch (KiCad schematic)
At the start: 20 parts, among them U2 LMV324

Commit message: Placement step 1: footprints in the PCB, grouped by function; zone sketch
- Footprints brought into the PCB through Konnect (KiCad 10 IPC) and sorted into
  function groups beside their boards (design/groups.py, stage_groups.py,
  tools/konnect_stage.py), plus 8 optional standoff holes and group labels.
- Main-board zone sketch with area budgets for review (design/zone_sketch.py,
  out/zone-sketch.png).
- WIDTH moved to U1 so each CV quad carries one 1V/OCT channel (d).
- gen_sch.py: stable sheet/symbol UUIDs, so rebuilds keep PCB links.
- Both boards 2-layer (d); Konnect setup notes; CLAUDE.md: pin map follows
  the layout.

Co-Authored-By: Claude Opus 5.5 <noreply@anthropic.com>
Claude-Session: https://claude.ai/code/session_01Cf5qNBi3oNHhbCjPHvswth
Parts:
- removed unit 4 of U2
- added C20: 100n, filter-module:C_0603, symbol Device:C
- added U1: LMV324, filter-module:SOIC-14_3.9x8.65mm_Pitch1.27mm, symbol Amplifier_Operational:LMV324
Connections:
- net +3V3_A: now also C20.1, U1.4 (V+)
- net ADC_WIDTH: now also U1.14
- net GND: now also C20.2, U1.11 (V-), U1.12 (+)
- net at C11.1, R15.1, R16.1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: now also U1.13 (-)
Other:
- note added: "U1: LMV324, ADC stages"

Commit message: Placement step 4: U1 and its CV group; ADC pins re-matched to the placed chips
Re-match pending d's OK (d questioned doing it now): tools/rematch_adc.py,
pinmap ADC_UNIT/SEED_ADC, schematic rebuilt, firmware and placement docs
updated, PCB pads reassigned (U1 re-added: its unit A moved sheets).
WIDTH trace not drawn yet.

Co-Authored-By: Claude Opus 5.5 <noreply@anthropic.com>
Claude-Session: https://claude.ai/code/session_01Cf5qNBi3oNHhbCjPHvswth
Parts:
- removed unit 4 of U1
- added unit 1 of U1
Connections:
- net ADC_WIDTH: now also U1.1
- net GND: now also U1.3 (+)
- net at C11.1, R15.1, R16.1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: now also U1.2 (-)
Changed lines of the file:
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@@
 		(at 228.6 76.2 0)
 		(mirror x)
-		(unit 4)
+		(unit 1)
 		(exclude_from_sim no)
 		(in_bom yes)
@@
 			)
 		)
-		(pin "12"
+		(pin "1"
 		)
-		(pin "13"
+		(pin "2"
 		)
-		(pin "14"
+		(pin "3"
 		)
 		(instances
@@
 				(path "/2d3363f2-481d-573e-813e-0e55dd9cdd97/8e40b2c3-2b41-533a-9c82-023551050a03"
 					(reference "U1")
-					(unit 4)
+					(unit 1)
 				)
 			)
