File: pcb/machine-filter/main-cv-inputs-5-8.kicad_sch (KiCad schematic)
At the start: 18 parts, among them U1 LMV324

Commit message: Placement step 1: footprints in the PCB, grouped by function; zone sketch
- Footprints brought into the PCB through Konnect (KiCad 10 IPC) and sorted into
  function groups beside their boards (design/groups.py, stage_groups.py,
  tools/konnect_stage.py), plus 8 optional standoff holes and group labels.
- Main-board zone sketch with area budgets for review (design/zone_sketch.py,
  out/zone-sketch.png).
- WIDTH moved to U1 so each CV quad carries one 1V/OCT channel (d).
- gen_sch.py: stable sheet/symbol UUIDs, so rebuilds keep PCB links.
- Both boards 2-layer (d); Konnect setup notes; CLAUDE.md: pin map follows
  the layout.

Co-Authored-By: Claude Opus 5.5 <noreply@anthropic.com>
Claude-Session: https://claude.ai/code/session_01Cf5qNBi3oNHhbCjPHvswth
Parts:
- removed C20: 100n, filter-module:C_0603, symbol Device:C
- removed unit 4 of U1
- removed unit 5 of U1
- added U2: LMV324, filter-module:SOIC-14_3.9x8.65mm_Pitch1.27mm, symbol Amplifier_Operational:LMV324
Connections:
- net ADC_EQF: now also U2.14
- net GND: now also U2.12 (+)
- net at C14.1, R26.2, R27.1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: now also U2.13 (-)
Other:
- note removed: "Op-amp supplies"
- note removed: "U1: LMV324, ADC stages"

Commit message: Placement step 4: U1 and its CV group; ADC pins re-matched to the placed chips
Re-match pending d's OK (d questioned doing it now): tools/rematch_adc.py,
pinmap ADC_UNIT/SEED_ADC, schematic rebuilt, firmware and placement docs
updated, PCB pads reassigned (U1 re-added: its unit A moved sheets).
WIDTH trace not drawn yet.

Co-Authored-By: Claude Opus 5.5 <noreply@anthropic.com>
Claude-Session: https://claude.ai/code/session_01Cf5qNBi3oNHhbCjPHvswth
Parts:
- removed unit 1 of U1
- added unit 4 of U1
Connections:
- net ADC_EQG: now also U1.7
- net ADC_SRR: now also U1.14; no longer U1.7
- net GND: now also U1.12 (+)
- net at C17.1, R38.2, R39.1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: now also U1.13 (-); no longer U1.6 (-)
- net at C15.1, R30.2, R31.1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: now also U1.6 (-)
Other:
- moved on the sheet: U1B
Changed lines of the file:
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@@
 		(at 228.6 76.2 0)
 		(mirror x)
-		(unit 1)
+		(unit 2)
 		(exclude_from_sim no)
 		(in_bom yes)
@@
 			)
 		)
-		(pin "1"
-		)
-		(pin "2"
-		)
-		(pin "3"
+		(pin "5"
+		)
+		(pin "6"
+		)
+		(pin "7"
 		)
 		(instances
@@
 				(path "/2d3363f2-481d-573e-813e-0e55dd9cdd97/3dd72cb2-cdc5-5f7b-b550-d0ad4f67f81a"
 					(reference "U1")
-					(unit 1)
+					(unit 2)
 				)
 			)
@@
 		(at 228.6 167.64 0)
 		(mirror x)
-		(unit 2)
+		(unit 4)
 		(exclude_from_sim no)
 		(in_bom yes)
@@
 			)
 		)
-		(pin "5"
-		)
-		(pin "6"
-		)
-		(pin "7"
+		(pin "12"
+		)
+		(pin "13"
+		)
+		(pin "14"
 		)
 		(instances
@@
 				(path "/2d3363f2-481d-573e-813e-0e55dd9cdd97/3dd72cb2-cdc5-5f7b-b550-d0ad4f67f81a"
 					(reference "U1")
-					(unit 2)
-				)
-			)
+					(unit 4)
+				)
+			)
