File: pcb/machine-filter/machine-filter.kicad_sch (KiCad schematic)
At the start: 0 parts

Commit message: Control chips placed; board-to-board connectors found by search: 4 lines (22+3+5+3 pins, 12 ground)
connector_search.py: lines live in legal straight runs on both boards (courtyard polygons, socket body and its
courtyard, leads under bodies), d's ground rules plus a ground on every connector; simulated annealing, 12
restarts. sync_headers.py deletes and re-adds the header footprints from the schematic, places both boards and
checks every pin pair lines up. auto_place.py now keeps other parts' leads out from under a body (U6 had RV4's
lead under it). Mux channels and LED sections re-checked: already shortest. Build OK, raw DRC: no real problems.

Co-Authored-By: Claude Opus 5.5 <noreply@anthropic.com>
Claude-Session: https://claude.ai/code/session_01Cf5qNBi3oNHhbCjPHvswth
Other:
- note added: "-10 V reference U5, expansion header J14, optional microSD J15 (DNP). Front: male headers JB1 (22 pins), JB2 (3 pins), JB3 (5 pins), JB4 (3 pins)."
- note added: "JA1, JA2, JA3, JA4"
- note added: "JB1, JB2, JB3, JB4"
- note added: "through-hole resistors and capacitors, female headers JA1, JA2, JA3, JA4."
- note removed: "-10 V reference U5, expansion header J14, optional microSD J15 (DNP). Front: male headers JB1 (15 pins), JB2 (13 pins), JB3 (10 pins)."
- note removed: "JA1, JA2, JA3"
- note removed: "JB1, JB2, JB3"
- note removed: "through-hole resistors and capacitors, female headers JA1, JA2, JA3."
Changed lines of the file:
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@@
 		)
 	)
-	(text "-10 V reference U5, expansion header J14, optional microSD J15 (DNP). Front: male headers JB1 (15 pins), JB2 (13 pins), JB3 (10 pins)."
+	(text "-10 V reference U5, expansion header J14, optional microSD J15 (DNP). Front: male headers JB1 (22 pins), JB2 (3 pins), JB3 (5 pins), JB4 (3 pins)."
 		(exclude_from_sim no)
 		(at 20.32 57.79 0)
@@
 		)
 	)
-	(text "through-hole resistors and capacitors, female headers JA1, JA2, JA3."
+	(text "through-hole resistors and capacitors, female headers JA1, JA2, JA3, JA4."
 		(exclude_from_sim no)
 		(at 20.32 71.13 0)
@@
 		)
 	)
-	(text "JB1, JB2, JB3"
+	(text "JB1, JB2, JB3, JB4"
 		(exclude_from_sim no)
 		(at 340.36 139.7 0)
@@
 		)
 	)
-	(text "JA1, JA2, JA3"
+	(text "JA1, JA2, JA3, JA4"
 		(exclude_from_sim no)
 		(at 276.86 198.12 0)

Commit message: Hand-soldering clearance (d: 1.25 mm): connectors re-searched, control parts re-placed
connector_search.py: header pads keep 1.25 mm from every other pad on both boards and from the whole box around
each jack, pot and LED (taken from the square pin-1 pad); --free leaves parts to be re-placed out of the search.
auto_place.py: control-board through-hole pads and anything near a header keep 1.25 mm; --free re-places parts.
Result: 3 lines, 30 + 5 + 2 pins (16 ground); the connector beside pot RV5 and the one between two CV jacks are
gone. Measured: nearest header-pad gap 1.35 mm, header to a body box 1.31 mm. Raw DRC: no real problems.

Co-Authored-By: Claude Opus 5.5 <noreply@anthropic.com>
Claude-Session: https://claude.ai/code/session_01Cf5qNBi3oNHhbCjPHvswth
Other:
- note added: "-10 V reference U5, expansion header J14, optional microSD J15 (DNP). Front: male headers JB1 (30 pins), JB2 (5 pins), JB3 (2 pins)."
- note added: "JA1, JA2, JA3"
- note added: "JB1, JB2, JB3"
- note added: "through-hole resistors and capacitors, female headers JA1, JA2, JA3."
- note removed: "-10 V reference U5, expansion header J14, optional microSD J15 (DNP). Front: male headers JB1 (22 pins), JB2 (3 pins), JB3 (5 pins), JB4 (3 pins)."
- note removed: "JA1, JA2, JA3, JA4"
- note removed: "JB1, JB2, JB3, JB4"
- note removed: "through-hole resistors and capacitors, female headers JA1, JA2, JA3, JA4."
Changed lines of the file:
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@@
 		)
 	)
-	(text "-10 V reference U5, expansion header J14, optional microSD J15 (DNP). Front: male headers JB1 (22 pins), JB2 (3 pins), JB3 (5 pins), JB4 (3 pins)."
+	(text "-10 V reference U5, expansion header J14, optional microSD J15 (DNP). Front: male headers JB1 (30 pins), JB2 (5 pins), JB3 (2 pins)."
 		(exclude_from_sim no)
 		(at 20.32 57.79 0)
@@
 		)
 	)
-	(text "through-hole resistors and capacitors, female headers JA1, JA2, JA3, JA4."
+	(text "through-hole resistors and capacitors, female headers JA1, JA2, JA3."
 		(exclude_from_sim no)
 		(at 20.32 71.13 0)
@@
 		)
 	)
-	(text "JB1, JB2, JB3, JB4"
+	(text "JB1, JB2, JB3"
 		(exclude_from_sim no)
 		(at 340.36 139.7 0)
@@
 		)
 	)
-	(text "JA1, JA2, JA3, JA4"
+	(text "JA1, JA2, JA3"
 		(exclude_from_sim no)
 		(at 276.86 198.12 0)

Commit message: Experiment (not chosen): connectors searched with a strict Seed-pocket rule; routing tool runs
The board now holds the pocket-rule connectors (4 lines, 34 pins) as an experiment; c08-handsolder (3 lines,
routed: main 5 unrouted / 61 vias, control 2 unrouted / 16 vias, DRC 0) stays the best candidate. route_board.py:
Freerouting 2.3 ignores direction costs from DSN, CLI and freerouting.json (tested); 90-degree snap works.
Paused for d: the header loop is repeating (post-mortem 2026-10-06).

Co-Authored-By: Claude Opus 5.5 <noreply@anthropic.com>
Claude-Session: https://claude.ai/code/session_01Cf5qNBi3oNHhbCjPHvswth
Other:
- note added: "-10 V reference U5, expansion header J14, optional microSD J15 (DNP). Front: male headers JB1 (7 pins), JB2 (11 pins), JB3 (7 pins), JB4 (9 pins)."
- note added: "JA1, JA2, JA3, JA4"
- note added: "JB1, JB2, JB3, JB4"
- note added: "through-hole resistors and capacitors, female headers JA1, JA2, JA3, JA4."
- note removed: "-10 V reference U5, expansion header J14, optional microSD J15 (DNP). Front: male headers JB1 (30 pins), JB2 (5 pins), JB3 (2 pins)."
- note removed: "JA1, JA2, JA3"
- note removed: "JB1, JB2, JB3"
- note removed: "through-hole resistors and capacitors, female headers JA1, JA2, JA3."
Changed lines of the file:
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@@
 		)
 	)
-	(text "-10 V reference U5, expansion header J14, optional microSD J15 (DNP). Front: male headers JB1 (30 pins), JB2 (5 pins), JB3 (2 pins)."
+	(text "-10 V reference U5, expansion header J14, optional microSD J15 (DNP). Front: male headers JB1 (7 pins), JB2 (11 pins), JB3 (7 pins), JB4 (9 pins)."
 		(exclude_from_sim no)
 		(at 20.32 57.79 0)
@@
 		)
 	)
-	(text "through-hole resistors and capacitors, female headers JA1, JA2, JA3."
+	(text "through-hole resistors and capacitors, female headers JA1, JA2, JA3, JA4."
 		(exclude_from_sim no)
 		(at 20.32 71.13 0)
@@
 		)
 	)
-	(text "JB1, JB2, JB3"
+	(text "JB1, JB2, JB3, JB4"
 		(exclude_from_sim no)
 		(at 340.36 139.7 0)
@@
 		)
 	)
-	(text "JA1, JA2, JA3"
+	(text "JA1, JA2, JA3, JA4"
 		(exclude_from_sim no)
 		(at 276.86 198.12 0)
